File: hardware/electronics/daughter-boards-v0.2/ui-panel-v0.2.kicad_pcb (KiCad board)
At the start: 2 copper layers, 58 x 28 mm, 13 parts

Commit message: ✨ 完善面板接口对齐与打印预览
Parts:
- removed the D_BAT at (40.0, 13.0)
- removed the D_STATUS at (34.0, 13.0)
- removed the J_USB_PANEL at (44.0, 24.0)
- removed the SW_MODE at (45.0, 18.0)
- removed the SW_START at (34.0, 18.0)
- added D_BAT: LED_BATTERY_0603_YELLOW, LED_0603_1608Metric, F.Cu at (32.0, 25.0)
- added D_STATUS: LED_STATUS_0603_GREEN, LED_0603_1608Metric, F.Cu at (29.0, 3.00)
- added J_USB_PANEL: USB-C_VERTICAL_16P_DIRECT, USB_C_Receptacle_G-Switch_GT-USB-7051x, F.Cu at (47.0, 26.0)
- added SW_MODE: SEALED_SMD_TACTILE_MODE, SW_SPST_TS-1088-xR020, F.Cu at (10.0, 20.0)
- added SW_START: SEALED_SMD_TACTILE_START, SW_SPST_TS-1088-xR020, F.Cu at (10.0, 8.00)
- J_OLED: value MX1.25_I2C_OLED_RESERVE_4P -> MX1.25_I2C_OLED_FPC_4P
- moved J_BUZ 15.1 mm to (38.0, 16.0)
- moved J_MOTHER 10.0 mm to (18.0, 17.0)
Other:
- board text added: "SEALED PANEL: OLED CABLE / DIRECT BTN / LED / USB-C"
- board text added: "USB-C 16P / PORT TO y+ BEZEL"
- board text removed: "D_BAT"
- board text removed: "D_STATUS"
- board text removed: "J_USB_PANEL"
- board text removed: "SEALED PANEL: OLED / BTN / LED / AUDIO"
- board text removed: "SW_MODE"
- board text removed: "SW_START"
- board text removed: "USB-C BULKHEAD + SILICONE CAP"
