File: hardware/electronics/daughter-boards-v0.2/ui-panel-v0.2.kicad_pcb (KiCad board)
At the start: 2 copper layers, 58 x 28 mm, 13 parts

Commit message: 🔌 统一 Type-C 充电入口
Parts:
- added R_CC1: 5k1 USB-C CC1 Rd, , F.Cu at (37.0, 3.00)
- added R_CC2: 5k1 USB-C CC2 Rd, , F.Cu at (41.0, 3.00)
- J_MOTHER: value MX1.25_MOTHER_UI_LOCK_12P -> MX1.25_MOTHER_UI_LOCK_14P_CHARGE
- J_USB_PANEL: value USB-C_VERTICAL_16P_DIRECT -> USB-C_VERTICAL_CHARGE_ONLY
Connections:
- J_USB_PANEL pad A6: usb_dp -> (no net)
- J_USB_PANEL pad A7: usb_dn -> (no net)
- J_USB_PANEL pad A8: usb_sbu2 -> (no net)
- J_USB_PANEL pad B6: usb_dp -> (no net)
- J_USB_PANEL pad B7: usb_dn -> (no net)
- J_USB_PANEL pad B8: usb_sbu1 -> (no net)
Other:
- board text added: "R_CC1"
- board text added: "R_CC2"
- board text added: "SEALED PANEL: OLED CABLE / DIRECT BTN / LED / CHARGE-ONLY USB-C"
- board text added: "USB-C CHARGE / VBUS-GND VIA J_MOTHER 14P"
- board text removed: "SEALED PANEL: OLED CABLE / DIRECT BTN / LED / USB-C"
- board text removed: "USB-C 16P / PORT TO y+ BEZEL"

Commit message: 🔌 修复线束契约与电子机械干涉
Parts:
- removed the J_USB_PANEL at (47.0, 26.0)
- added J_USB_PANEL: USB-C_VERTICAL_CHARGE_ONLY, USB_C_Receptacle_GCT_USB4105-xx-A_16P_TopMnt_Horizontal, F.Cu at (47.2, 24.8)
- moved J_MOTHER 5.50 mm to (23.5, 17.0)
