File: hardware/electronics/esp32-control-v0.1/esp32-control-v0.1.kicad_pcb (KiCad board)
At the start: 2 copper layers, 86 x 32 mm, 43 parts, among them J1 USB-C-POWER-DATA, J2 MX1.25_PROTECTED_1S_BAT, J3 MX1.25_SENSOR_10-30V_IN, J4 MX1.25_M6_CARRIER_HOST, J5 MX1.25_PVDF_ADC_AUX, J6 MX1.25_PVDF_CMP_AUX_DNP, J7 MX1.25_UI_PANEL_LOCK_12P, J8 MX1.25_M6_SENSOR_RAIL_LINK, SW1 IP5305 KEY, U1 ESP32-S3-WROOM-1-N16R8, U2 IP5305T-HSOP8-1EP, U3 TPS62162-QFN8-EP

Commit message: 🔌 统一 Type-C 充电入口
Parts:
- removed J1: USB-C-POWER-DATA, 
- removed R1: 22R USB_DP, 
- removed R2: 22R USB_DN, 
- removed R3: 5k1 CC1, 
- removed R4: 5k1 CC2, 
- J7: value MX1.25_UI_PANEL_LOCK_12P -> MX1.25_UI_PANEL_LOCK_14P_CHARGE
Connections:
- U1 pad 14: usb_dn_mcu -> (no net)
- U1 pad 15: usb_dp_mcu -> (no net)
Other:
- board text added: "J7: UI LOCK 14P / VBUS GND"
- board text removed: "J1"
- board text removed: "J7: UI LOCK 12P"
- board text removed: "R1"
- board text removed: "R2"
- board text removed: "R3"
- board text removed: "R4"

Commit message: 🔧 修正 ESP32 原生封装与焊盘装配
Parts:
- U1: footprint (none) -> ESP32-S3-WROOM-1
- turned U1 to 90 degrees
Other:
- board text removed: "U1 ESP32-S3"

Commit message: 🔌 修复线束契约与电子机械干涉
Parts:
- moved H1 43.2 mm to (55.0, 16.0)
- moved F1 20.0 mm to (35.0, 3.80)
Connections:
- D2 pad 2: gnd -> sensor_gnd
- J3 pad 2: gnd -> sensor_gnd
- J8 pad 2: gnd -> sensor_gnd
